Commit message: Changed the hardware interface from position_constrollers to effort_controllers.

File: robotic_arm_description/urdf/forearm.xacro (robot description, xacro)
@@ -57,5 +57,5 @@
     <origin rpy=" 0 0 0" xyz="0 0 0.035 " />
     <axis xyz="0 0 1" />
-    <limit effort="10000" lower="-3e+307" upper="3e+307" velocity="100" />
+    <limit effort="100000" lower="-3e+307" upper="3e+307" velocity="100" />
   </joint>
   <joint name="forearm_0_1_joint" type="revolute">
@@ -64,5 +64,5 @@
     <origin rpy=" 0 0 0" xyz="0 0 0.09 " />
     <axis xyz="0 1 0" />
-    <limit effort="10000" lower="-2.3" upper="2.3" velocity="100" />
+    <limit effort="100000" lower="-2.3" upper="2.3" velocity="100" />
   </joint>
   <joint name="forearm_1_2_joint" type="fixed">

File: robotic_arm_description/urdf/transmission.xacro (robot description, xacro)
@@ -5,8 +5,8 @@
         <type>transmission_interface/SimpleTransmission</type>
         <joint name="base_forearm_joint">
-            <hardwareInterface>hardware_interface/PositionJointInterface</hardwareInterface>
+            <hardwareInterface>hardware_interface/EffortJointInterface</hardwareInterface>
         </joint>
         <actuator name="base_forearm_joint_motor">
-            <hardwareInterface>hardware_interface/PositionJointInterface</hardwareInterface>
+            <hardwareInterface>hardware_interface/EffortJointInterface</hardwareInterface>
             <mechanicalReduction>1</mechanicalReduction>
         </actuator>
@@ -15,18 +15,8 @@
         <type>transmission_interface/SimpleTransmission</type>
         <joint name="forearm_0_1_joint">
-            <hardwareInterface>hardware_interface/PositionJointInterface</hardwareInterface>
+            <hardwareInterface>hardware_interface/EffortJointInterface</hardwareInterface>
         </joint>
         <actuator name="forearm_0_1_joint_motor">
-            <hardwareInterface>hardware_interface/PositionJointInterface</hardwareInterface>
-            <mechanicalReduction>1</mechanicalReduction>
-        </actuator>
-    </transmission>
-    <transmission name="trans_forearm_gripper_joint">
-        <type>transmission_interface/SimpleTransmission</type>
-        <joint name="forearm_gripper_joint">
-            <hardwareInterface>hardware_interface/PositionJointInterface</hardwareInterface>
-        </joint>
-        <actuator name="forearm_gripper_joint_motor">
-            <hardwareInterface>hardware_interface/PositionJointInterface</hardwareInterface>
+            <hardwareInterface>hardware_interface/EffortJointInterface</hardwareInterface>
             <mechanicalReduction>1</mechanicalReduction>
         </actuator>
