Commit message: Planning groups merged into one.

File: robotic_arm_description/urdf/arm.xacro (robot description, xacro)
@@ -64,5 +64,5 @@
     <origin rpy=" 0 0 0" xyz="0 0 0.09 " />
     <axis xyz="0 1 0" />
-    <limit effort="100000" lower="-2.3" upper="2.3" velocity="100" />
+    <limit effort="100000" lower="-1.8" upper="1.8" velocity="100" />
   </joint>
   <joint name="arm_1_2_joint" type="fixed">

File: robotic_arm_description/urdf/forearm.xacro (robot description, xacro)
@@ -64,5 +64,5 @@
     <origin rpy=" 0 0 0" xyz="0 0 0.09 " />
     <axis xyz="0 1 0" />
-    <limit effort="100000" lower="-2.3" upper="2.3" velocity="100" />
+    <limit effort="1000000" lower="-1.8" upper="1.8" velocity="100" />
   </joint>
   <joint name="forearm_1_2_joint" type="fixed">

Commit message: Modified joint limits.

File: robotic_arm_description/urdf/arm.xacro (robot description, xacro)
@@ -64,5 +64,5 @@
     <origin rpy=" 0 0 0" xyz="0 0 0.09 " />
     <axis xyz="0 1 0" />
-    <limit effort="100000" lower="-1.8" upper="1.8" velocity="100" />
+    <limit effort="100000" lower="-1.4" upper="1.4" velocity="100" />
   </joint>
   <joint name="arm_1_2_joint" type="fixed">

File: robotic_arm_description/urdf/forearm.xacro (robot description, xacro)
@@ -64,5 +64,5 @@
     <origin rpy=" 0 0 0" xyz="0 0 0.09 " />
     <axis xyz="0 1 0" />
-    <limit effort="1000000" lower="-1.8" upper="1.8" velocity="100" />
+    <limit effort="1000000" lower="-1.4" upper="1.4" velocity="100" />
   </joint>
   <joint name="forearm_1_2_joint" type="fixed">
