Commit message: Robotic arm now consists of 2 arms.

File: robotic_arm_description/urdf/gazebo.xacro (robot description, xacro)
@@ -7,7 +7,4 @@
         </plugin>
     </gazebo>
-    <gazebo reference="forearm_1_2_joint">
-        <disableFixedJointLumping>true</disableFixedJointLumping>
-    </gazebo>
     <gazebo reference="base_link">
         <static>true</static>
@@ -16,5 +13,11 @@
         <disableFixedJointLumping>true</disableFixedJointLumping>
     </gazebo>
-    <gazebo reference="forearm_gripper_joint">
+    <gazebo reference="forearm_1_2_joint">
+        <disableFixedJointLumping>true</disableFixedJointLumping>
+    </gazebo>
+    <gazebo reference="arm_1_2_joint">
+        <disableFixedJointLumping>true</disableFixedJointLumping>
+    </gazebo>
+    <gazebo reference="arm_gripper_joint">
         <disableFixedJointLumping>true</disableFixedJointLumping>
     </gazebo>

File: robotic_arm_description/urdf/gripper.xacro (robot description, xacro)
@@ -20,6 +20,6 @@
     </collision>
   </link>
-  <joint name="forearm_gripper_joint" type="fixed">
-    <parent link="forearm_2_link" />
+  <joint name="arm_gripper_joint" type="fixed">
+    <parent link="arm_2_link" />
     <child link="gripper_link" />
     <origin rpy=" 0 0 0" xyz="0 0 0.42 " />

File: robotic_arm_description/urdf/robotic_arm_simulator.xacro (robot description, xacro)
@@ -5,4 +5,5 @@
     <xacro:include filename="$(find robotic_arm_description)/urdf/base.xacro" />
     <xacro:include filename="$(find robotic_arm_description)/urdf/forearm.xacro" />
+    <xacro:include filename="$(find robotic_arm_description)/urdf/arm.xacro" />
     <xacro:include filename="$(find robotic_arm_description)/urdf/gripper.xacro" />
     <xacro:include filename="$(find robotic_arm_description)/urdf/gazebo.xacro" />

File: robotic_arm_description/urdf/transmission.xacro (robot description, xacro)
@@ -22,3 +22,24 @@
         </actuator>
     </transmission>
+    <!-- ARM -->
+    <transmission name="trans_forearm_arm_joint">
+        <type>transmission_interface/SimpleTransmission</type>
+        <joint name="forearm_arm_joint">
+            <hardwareInterface>hardware_interface/EffortJointInterface</hardwareInterface>
+        </joint>
+        <actuator name="forearm_arm_joint_motor">
+            <hardwareInterface>hardware_interface/EffortJointInterface</hardwareInterface>
+            <mechanicalReduction>1</mechanicalReduction>
+        </actuator>
+    </transmission>
+    <transmission name="trans_arm_0_1_joint">
+        <type>transmission_interface/SimpleTransmission</type>
+        <joint name="arm_0_1_joint">
+            <hardwareInterface>hardware_interface/EffortJointInterface</hardwareInterface>
+        </joint>
+        <actuator name="arm_0_1_joint_motor">
+            <hardwareInterface>hardware_interface/EffortJointInterface</hardwareInterface>
+            <mechanicalReduction>1</mechanicalReduction>
+        </actuator>
+    </transmission>
 </robot>

Commit message: Gripper link can now rotate around one axis.

File: robotic_arm_description/urdf/gazebo.xacro (robot description, xacro)
@@ -19,6 +19,3 @@
         <disableFixedJointLumping>true</disableFixedJointLumping>
     </gazebo>
-    <gazebo reference="arm_gripper_joint">
-        <disableFixedJointLumping>true</disableFixedJointLumping>
-    </gazebo>
 </robot>

File: robotic_arm_description/urdf/gripper.xacro (robot description, xacro)
@@ -20,8 +20,10 @@
     </collision>
   </link>
-  <joint name="arm_gripper_joint" type="fixed">
+  <joint name="arm_gripper_joint" type="revolute">
     <parent link="arm_2_link" />
     <child link="gripper_link" />
     <origin rpy=" 0 0 0" xyz="0 0 0.42 " />
+    <axis xyz="0 0 1" />
+    <limit effort="100000" lower="-3e+150" upper="3e+150" velocity="100" />
   </joint>
 </robot>

File: robotic_arm_description/urdf/transmission.xacro (robot description, xacro)
@@ -43,3 +43,14 @@
         </actuator>
     </transmission>
+    <!-- GRIPPER -->
+    <transmission name="trans_arm_gripper_joint">
+        <type>transmission_interface/SimpleTransmission</type>
+        <joint name="arm_gripper_joint">
+            <hardwareInterface>hardware_interface/EffortJointInterface</hardwareInterface>
+        </joint>
+        <actuator name="arm_gripper_joint_motor">
+            <hardwareInterface>hardware_interface/EffortJointInterface</hardwareInterface>
+            <mechanicalReduction>1</mechanicalReduction>
+        </actuator>
+    </transmission>
 </robot>
